File: night-light-charger.kicad_pcb (KiCad board)
At the start: 2 copper layers, 40 x 28 mm, 21 parts, among them J1 USB_C_Receptacle_PowerOnly_6P, Q1 IRLML2803, U1 BQ25172DSGR

Commit message: Update part information
Parts:
- removed REF**: OSHW-Logo2_7.3x6mm_SilkScreen, Symbol:OSHW-Logo2_7.3x6mm_SilkScreen
- removed REF**: KiCad-Logo2_5mm_SilkScreen, Symbol:KiCad-Logo2_5mm_SilkScreen
