File: night-light-charger.kicad_sch (KiCad schematic)
At the start: 19 parts, among them J1 USB_C_Receptacle_PowerOnly_6P, Q1 IRLML2803, U1 BQ25172DSGR

Commit message: Update part information
Parts:
- BT1, TP1, TP2, TP3: now left out of the parts list
- D3: MPN (none) -> LTST-S326KGJRKT
- J1: MPN (none) -> GT-USB-7010ASV
- Q1: MPN (none) -> IRLML2803TRPBF
- RV1: MPN (none) -> 3224W-1-203E
- TH1: MPN (none) -> MF52A103J3435 (A1)
- U1: MPN (none) -> BQ25172DSGR
Changed lines of the file:
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@@
+			)
+		)
+		(property "MPN" "BQ25172DSGR"
+			(at 88.9 44.45 0)
+			(effects
+				(font
+					(size 1.27 1.27)
+				)
+				(hide yes)
 			)
 		)
@@
 			)
 		)
+		(property "MPN" "MF52A103J3435 (A1) "
+			(at 69.85 74.93 0)
+			(effects
+				(font
+					(size 1.27 1.27)
+				)
+				(hide yes)
+			)
+		)
 		(pin "1"
 		)
@@
 		(unit 1)
 		(exclude_from_sim no)
-		(in_bom yes)
+		(in_bom no)
 		(on_board yes)
 		(dnp no)
@@
 			)
 		)
+		(property "MPN" "IRLML2803TRPBF"
+			(at 160.02 74.93 0)
+			(effects
+				(font
+					(size 1.27 1.27)
+				)
+				(hide yes)
+			)
+		)
 		(pin "2"
 		)
@@
 			)
 		)
+		(property "MPN" "LTST-S326KGJRKT"
+			(at 160.02 62.23 90)
+			(effects
+				(font
+					(size 1.27 1.27)
+				)
+				(hide yes)
+			)
+		)
 		(pin "2"
 		)
@@
 		(unit 1)
 		(exclude_from_sim no)
-		(in_bom yes)
+		(in_bom no)
 		(on_board yes)
 		(dnp no)
@@
 		(unit 1)
 		(exclude_from_sim no)
-		(in_bom yes)
+		(in_bom no)
 		(on_board yes)
 		(dnp no)
@@
 			)
 		)
+		(property "MPN" "3224W-1-203E"
+			(at 77.47 64.77 0)
+			(effects
+				(font
+					(size 1.27 1.27)
+				)
+				(hide yes)
+			)
+		)
 		(pin "1"
 		)
@@
 		(unit 1)
 		(exclude_from_sim no)
-		(in_bom yes)
+		(in_bom no)
 		(on_board yes)
 		(dnp no)
@@
 			(at 31.75 52.07 0)
 			(effects
+				(font
+					(size 1.27 1.27)
+				)
+				(hide yes)
+			)
+		)
+		(property "MPN" "GT-USB-7010ASV"
+			(at 31.75 52.07 0)
+			(effects
